Commit message: update ur10e

File: genesis/assets/urdf/ur10e/robot_wsg50.urdf (robot description, URDF)
Before this commit: robot ur10e_robot, 12 links, 11 joints
Links:
- added link camera_1_link; collision box size=0.05 0.05 0.02; visual box size=0.05 0.05 0.02
Joints:
- added joint camera_1_joint: type fixed, parent wrist_3_link, child camera_1_link

Commit message: camera ready

File: genesis/assets/urdf/ur10e/robot_wsg50.urdf (robot description, URDF)
Before this commit: robot ur10e_robot, 13 links, 12 joints
Links:
- removed link camera_1_link
- added link camera_wrist_back_link
- added link camera_wrist_link
Joints:
- removed joint camera_1_joint
- added joint camera_wrist_back_joint: type fixed, parent wrist_3_link, child camera_wrist_back_link, origin xyz=0 -0.14 0 rpy=0.7853 -3.14 0
- added joint camera_wrist_joint: type fixed, parent wrist_3_link, child camera_wrist_link, origin xyz=0 0.14 0 rpy=-2.35619445 0 0
